Commit message: feat: added accelerometer frames to urdfs

File: robots/common/franka_arm.xacro (robot description, xacro)
@@ -8,7 +8,8 @@
   <!-- inertials: description of the inertials that comes from a YAML file. Example definition: ${xacro.load_yaml('$(find franka_description)/robots/fr3/inertials.yaml')} -->
   <!-- dynamics: description of the dynamics that comes from a YAML file. Example definition: ${xacro.load_yaml('$(find franka_description)/robots/fr3/dynamics.yaml')} -->
-  <xacro:macro name="franka_arm" params="arm_id arm_prefix:='' no_prefix:=false description_pkg:='franka_description' connected_to:='base' xyz:='0 0 0' rpy:='0 0 0' gazebo:='false' safety_distance:=0 joint_limits inertials kinematics dynamics with_sc:=false" >
+  <xacro:macro name="franka_arm" params="arm_id arm_prefix:='' no_prefix:=false description_pkg:='franka_description' connected_to:='base' xyz:='0 0 0' rpy:='0 0 0' gazebo:='false' safety_distance:=0 joint_limits inertials kinematics accelerometer_config dynamics with_sc:=false" >
     <!-- Define a property that defaults to 'arm_prefix_arm_id' concatenated with an underscore if 'no_prefix' is not set -->
     <xacro:property name="prefix" value="${'' if no_prefix else arm_prefix + arm_id + '_'}" />
+    <xacro:property name="with_accelerometers" value="${'false' if accelerometer_config == 'none' else 'true'}" />
     <xacro:if value="${gazebo}">
       <xacro:property name="connected_to" value="" />
@@ -23,10 +24,10 @@
       </joint>
     </xacro:unless>
-    <xacro:link_with_sc no_prefix="${no_prefix}" name="link0" gazebo="${gazebo}" with_sc="${with_sc}">
+    <xacro:link_with_sc no_prefix="${no_prefix}" name="link0" gazebo="${gazebo}" with_sc="${with_sc}" with_accelerometers="${with_accelerometers}">
       <self_collision_geometries>
         <xacro:collision_capsule xyz="-0.075 0 0.06" direction="x" radius="${0.06+safety_distance}" length="0.03" />
       </self_collision_geometries>
     </xacro:link_with_sc>
-    <xacro:link_with_sc no_prefix="${no_prefix}" name="link1" gazebo="${gazebo}" with_sc="${with_sc}">
+    <xacro:link_with_sc no_prefix="${no_prefix}" name="link1" gazebo="${gazebo}" with_sc="${with_sc}" with_accelerometers="${with_accelerometers}">
       <self_collision_geometries>
         <xacro:collision_capsule xyz="0 0 -191.5e-3" radius="${0.06+safety_distance}" length="0.283" />
@@ -41,5 +42,5 @@
       <xacro:franka-dynamics name="joint1" config="${dynamics}" />
     </joint>
-    <xacro:link_with_sc no_prefix="${no_prefix}" name="link2" gazebo="${gazebo}" with_sc="${with_sc}">
+    <xacro:link_with_sc no_prefix="${no_prefix}" name="link2" gazebo="${gazebo}" with_sc="${with_sc}" with_accelerometers="${with_accelerometers}">
       <self_collision_geometries>
         <xacro:collision_capsule xyz="0 0 0" radius="${0.06+safety_distance}" length="0.12" />
@@ -54,5 +55,5 @@
       <xacro:franka-dynamics name="joint2" config="${dynamics}" />
     </joint>
-    <xacro:link_with_sc no_prefix="${no_prefix}" name="link3" gazebo="${gazebo}" with_sc="${with_sc}">
+    <xacro:link_with_sc no_prefix="${no_prefix}" name="link3" gazebo="${gazebo}" with_sc="${with_sc}" with_accelerometers="${with_accelerometers}">
       <self_collision_geometries>
         <xacro:collision_capsule xyz="0 0 -0.145" radius="${0.06+safety_distance}" length="0.15" />
@@ -67,5 +68,5 @@
       <xacro:franka-dynamics name="joint3" config="${dynamics}" />
     </joint>
-    <xacro:link_with_sc no_prefix="${no_prefix}" name="link4" gazebo="${gazebo}" with_sc="${with_sc}">
+    <xacro:link_with_sc no_prefix="${no_prefix}" name="link4" gazebo="${gazebo}" with_sc="${with_sc}" with_accelerometers="${with_accelerometers}">
       <self_collision_geometries>
         <xacro:collision_capsule xyz="0 0 0" radius="${0.06+safety_distance}" length="0.12" />
@@ -80,5 +81,5 @@
       <xacro:franka-dynamics name="joint4" config="${dynamics}" />
     </joint>
-    <xacro:link_with_sc no_prefix="${no_prefix}" name="link5" gazebo="${gazebo}" with_sc="${with_sc}">
+    <xacro:link_with_sc no_prefix="${no_prefix}" name="link5" gazebo="${gazebo}" with_sc="${with_sc}" with_accelerometers="${with_accelerometers}">
       <self_collision_geometries>
         <xacro:collision_capsule xyz="0 0 -0.26"    radius="${0.060+safety_distance}" length="0.10" />
@@ -94,5 +95,5 @@
       <xacro:franka-dynamics name="joint5" config="${dynamics}" />
     </joint>
-    <xacro:link_with_sc no_prefix="${no_prefix}" name="link6" gazebo="${gazebo}" with_sc="${with_sc}">
+    <xacro:link_with_sc no_prefix="${no_prefix}" name="link6" gazebo="${gazebo}" with_sc="${with_sc}" with_accelerometers="false">
       <self_collision_geometries>
         <xacro:collision_capsule xyz="0 0 -0.03" radius="${0.05+safety_distance}" length="0.08" />
@@ -107,5 +108,5 @@
       <xacro:franka-dynamics name="joint6" config="${dynamics}" />
     </joint>
-    <xacro:link_with_sc no_prefix="${no_prefix}" name="link7" gazebo="${gazebo}" rpy="0 0 ${pi/4}" with_sc="${with_sc}">
+    <xacro:link_with_sc no_prefix="${no_prefix}" name="link7" gazebo="${gazebo}" rpy="0 0 ${pi/4}" with_sc="${with_sc}" with_accelerometers="false">
       <self_collision_geometries>
         <xacro:collision_capsule xyz="0 0 0.01" direction="z" radius="${0.04+safety_distance}" length="0.14" />

File: robots/common/franka_robot.xacro (robot description, xacro)
@@ -5,4 +5,5 @@
                       joint_limits
                       kinematics
+                      accelerometer_config:=none
                       inertials
                       dynamics
@@ -41,4 +42,5 @@
       joint_limits="${joint_limits}"
       kinematics="${kinematics}"
+      accelerometer_config="${accelerometer_config}"
       inertials="${inertials}"
       dynamics="${dynamics}"

File: robots/common/utils.xacro (robot description, xacro)
@@ -32,5 +32,5 @@
   <!-- self_collision_geometries:  self <collision> models        -->
   <!-- ========================================================== -->
-  <xacro:macro name="link_with_sc" params="name no_prefix:='false' rpy:='0 0 0' **self_collision_geometries gazebo:=false with_sc:=false">
+  <xacro:macro name="link_with_sc" params="name no_prefix:='false' rpy:='0 0 0' **self_collision_geometries gazebo:=false with_sc:=false with_accelerometers:=false">
     <xacro:property name="prefix" value="${'' if no_prefix else arm_prefix + arm_id + '_'}" />
     <!-- sub-link defining detailed meshes for collision with environment -->
@@ -61,4 +61,7 @@
         <child link="${prefix}${name}_sc" />
       </joint>
+    </xacro:if>
+    <xacro:if value="${with_accelerometers}">
+      <xacro:franka-accelerometers prefix="${prefix}" name="${name}" config="${accelerometer_config}" />
     </xacro:if>
   </xacro:macro>
@@ -250,3 +253,30 @@
              xyz="${kinematics.x} ${kinematics.y} ${kinematics.z}" />
   </xacro:macro>
+  <!-- ================================================================================== -->
+  <!-- Adds the accelerometer frames given a config file of link accelerometers           -->
+  <!--                                                                                    -->
+  <!-- name   - Name of the link for which to add accelerometers to                       -->
+  <!-- prefix - Prefix to name                                                            -->
+  <!-- config - YAML struct defining link accelerometers (e.g. fr3v2/accelerometers.yaml) -->
+  <!-- ================================================================================== -->
+  <xacro:macro name="franka-accelerometers" params="name prefix config">
+      <xacro:property name="accelerometer_top" value="${config[name]['accelerometer_top']}" lazy_eval="false" />
+      <xacro:property name="accelerometer_bottom" value="${config[name]['accelerometer_bottom']}" lazy_eval="false" />
+      <link name="${prefix}${name}_accelerometer_top">
+      </link>
+      <joint name="${prefix}${name}_accelerometer_top_joint" type="fixed">
+        <origin rpy="${accelerometer_top.roll} ${accelerometer_top.pitch} ${accelerometer_top.yaw}"
+             xyz="${accelerometer_top.x} ${accelerometer_top.y} ${accelerometer_top.z}" />
+        <parent link="${prefix}${name}" />
+        <child link="${prefix}${name}_accelerometer_top" />
+      </joint>
+      <link name="${prefix}${name}_accelerometer_bottom">
+      </link>
+      <joint name="${prefix}${name}_accelerometer_bottom_joint" type="fixed">
+        <origin rpy="${accelerometer_bottom.roll} ${accelerometer_bottom.pitch} ${accelerometer_bottom.yaw}"
+             xyz="${accelerometer_bottom.x} ${accelerometer_bottom.y} ${accelerometer_bottom.z}" />
+        <parent link="${prefix}${name}" />
+        <child link="${prefix}${name}_accelerometer_bottom" />
+      </joint>
+  </xacro:macro>
 </robot>

File: robots/fp3/fp3.urdf.xacro (robot description, xacro)
@@ -51,4 +51,5 @@
                       inertials="${xacro.load_yaml('$(find franka_description)/robots/fp3/inertials.yaml')}"
                       kinematics="${xacro.load_yaml('$(find franka_description)/robots/fp3/kinematics.yaml')}"
+                      accelerometer_config="${xacro.load_yaml('$(find franka_description)/robots/fp3/accelerometers.yaml')}"
                       dynamics="${xacro.load_yaml('$(find franka_description)/robots/fp3/dynamics.yaml')}"
                       gazebo="$(arg gazebo)"

File: robots/fr3/fr3.urdf.xacro (robot description, xacro)
@@ -51,4 +51,5 @@
                       inertials="${xacro.load_yaml('$(find franka_description)/robots/fr3/inertials.yaml')}"
                       kinematics="${xacro.load_yaml('$(find franka_description)/robots/fr3/kinematics.yaml')}"
+                      accelerometer_config="${xacro.load_yaml('$(find franka_description)/robots/fr3/accelerometers.yaml')}"
                       dynamics="${xacro.load_yaml('$(find franka_description)/robots/fr3/dynamics.yaml')}"
                       gazebo="$(arg gazebo)"

File: robots/fr3_duo/fr3_duo_arm.urdf.xacro (robot description, xacro)
@@ -67,4 +67,5 @@
   <xacro:arg name="inertials_path" default="$(find franka_description)/robots/${arm_id_i}/inertials.yaml"/>
   <xacro:arg name="kinematics_path" default="$(find franka_description)/robots/${arm_id_i}/kinematics.yaml"/>
+  <xacro:arg name="accelerometers_path" default="$(find franka_description)/robots/${arm_id_i}/accelerometers.yaml"/>
   <xacro:arg name="dynamics_path" default="$(find franka_description)/robots/${arm_id_i}/dynamics.yaml"/>
   <xacro:arg name="joint_limits_path" default="$(find franka_description)/robots/${arm_id_i}/joint_limits.yaml"/>
@@ -73,4 +74,5 @@
                       inertials="${xacro.load_yaml('$(arg inertials_path)')}"
                       kinematics="${xacro.load_yaml('$(arg kinematics_path)')}"
+                      accelerometers="${xacro.load_yaml('$(arg accelerometers_path)')}"
                       dynamics="${xacro.load_yaml('$(arg dynamics_path)')}"
                       gazebo="$(arg gazebo)"

File: robots/fr3v2/fr3v2.urdf.xacro (robot description, xacro)
@@ -52,4 +52,5 @@
                       kinematics="${xacro.load_yaml('$(find franka_description)/robots/fr3v2/kinematics.yaml')}"
                       dynamics="${xacro.load_yaml('$(find franka_description)/robots/fr3v2/dynamics.yaml')}"
+                      accelerometer_config="${xacro.load_yaml('$(find franka_description)/robots/fr3v2/accelerometers.yaml')}"
                       gazebo="$(arg gazebo)"
                       hand="$(arg hand)"
