Commit message: fix: group definition checking for right tcp

File: end_effectors/franka_hand/franka_hand.srdf.xacro (robot description, xacro)
@@ -17,5 +17,5 @@
       <joint name="${prefix}finger_joint2" value="0"/>
     </group_state>
-    <end_effector name="${prefix}hand" parent_link="${prefix}link8" group="${prefix}hand" parent_group="${prefix}arm"/>
+    <end_effector name="${prefix}hand" parent_link="${prefix}hand_tcp" group="${prefix}hand" parent_group="${prefix}arm"/>
     <disable_collisions link1="${prefix}hand" link2="${prefix}leftfinger" reason="Adjacent"/>
     <disable_collisions link1="${prefix}hand" link2="${prefix}rightfinger" reason="Adjacent"/>

File: robots/common/franka_arm.srdf.xacro (robot description, xacro)
@@ -4,5 +4,6 @@
         <xacro:property name="prefix" value="${'' if no_prefix else arm_prefix + arm_id + '_'}" />
         <xacro:include filename="$(find franka_description)/robots/common/group_definition.xacro"/>
-        <xacro:group_definition prefix="${prefix}" group_name="${prefix}arm" tip_link="${prefix}link8"/>
+        <xacro:property name="tip_link" value="${prefix + 'hand_tcp' if hand and ee_id == 'franka_hand' else prefix + 'link8'}"/>
+        <xacro:group_definition prefix="${prefix}" group_name="${prefix}arm" tip_link="${tip_link}"/>
         <virtual_joint name="virtual_joint" type="fixed" parent_frame="world" child_link="base"/>
         <disable_collisions link1="${prefix}link0" link2="${prefix}link1" reason="Adjacent"/>
