Commit message: * Refactor FR3 Duo Robot Configuration
    - Removed the cover kinematics argument from fr3_duo.urdf.xacro as it is no longer needed.
    - Updated inertials.yaml for fr3_duo_cover and fr3_duo_mount to indicate that values need to be corrected.
    - Deleted the kinematics.yaml file for fr3_duo_cover since it is no longer in use.
    - Removed fr3_duo_fixed_structure.urdf.xacro as it is obsolete.
    - Adjusted kinematic parameters in fr3_duo_mount's kinematics.yaml for both left and right configurations to new values.

File: robots/fr3_duo/fr3_duo.urdf.xacro (robot description, xacro)
@@ -53,7 +53,6 @@
       <origin xyz="0 0 0" rpy="0 0 0" />
   </xacro:mount>
-  <xacro:arg name="cover_kinematics" default="$(find franka_description)/robots/fr3_duo/fr3_duo_cover/kinematics.yaml"/>
   <xacro:cover name="cover" parent="mount_link" inertials="${xacro.load_yaml('$(find franka_description)/robots/fr3_duo/fr3_duo_cover/inertials.yaml')}">
-      <origin xyz="0 0 0" rpy="0 0 0" />
+      <origin xyz="0 0 0.068" rpy="0 0 0" />
   </xacro:cover>
   <xacro:property name="number_of_robots" value = "2"/>
@@ -80,9 +79,11 @@
       <xacro:arg name="dynamics_path" default="$(find franka_description)/robots/${arm_id_i}/dynamics.yaml"/>
       <xacro:arg name="joint_limits_path" default="$(find franka_description)/robots/${arm_id_i}/joint_limits.yaml"/>
+      <xacro:arg name="accelerometers_path" default="$(find franka_description)/robots/${arm_id_i}/accelerometers.yaml"/>
       <xacro:franka_robot arm_id="${arm_id_i}"
                           joint_limits="${xacro.load_yaml('$(arg joint_limits_path)')}"
                           inertials="${xacro.load_yaml('$(arg inertials_path)')}"
-                          kinematics="${xacro.load_yaml('$(arg kinematics_path)')}"
+                          kinematics="${xacro.load_yaml('$(arg kinematics_path')}"
                           dynamics="${xacro.load_yaml('$(arg dynamics_path)')}"
+                          accelerometer_config="${xacro.load_yaml('$(arg accelerometers_path)')}"
                           gazebo="$(arg gazebo)"
                           hand="$(arg hand)"

File: robots/fr3_duo/fr3_duo_arm.urdf.xacro (robot description, xacro)
@@ -74,5 +74,5 @@
                       inertials="${xacro.load_yaml('$(arg inertials_path)')}"
                       kinematics="${xacro.load_yaml('$(arg kinematics_path)')}"
-                      accelerometers="${xacro.load_yaml('$(arg accelerometers_path)')}"
+                      accelerometer_config="${xacro.load_yaml('$(arg accelerometers_path)')}"
                       dynamics="${xacro.load_yaml('$(arg dynamics_path)')}"
                       gazebo="$(arg gazebo)"

File: robots/fr3_duo/fr3_duo_fixed_structure.urdf.xacro (robot description, xacro)
@@ -11,5 +11,5 @@
   <xacro:arg name="cover_kinematics" default="$(find franka_description)/robots/fr3_duo/fr3_duo_cover/kinematics.yaml"/>
   <xacro:cover name="cover" parent="mount_link" inertials="${xacro.load_yaml('$(find franka_description)/robots/fr3_duo/fr3_duo_cover/inertials.yaml')}">
-      <origin xyz="0 0 0" rpy="0 0 0" />
+      <origin xyz="0 0 0.068" rpy="0 0 0" />
   </xacro:cover>
 </robot>

Commit message: feat: mount and cover belong to the same link feat: updated inertials

File: robots/fr3_duo/fr3_duo.urdf.xacro (robot description, xacro)
@@ -3,5 +3,4 @@
   <xacro:include filename="$(find franka_description)/robots/common/franka_robot.xacro"/>
   <xacro:include filename="$(find franka_description)/robots/fr3_duo/fr3_duo_mount/fr3_duo_mount.xacro" />
-  <xacro:include filename="$(find franka_description)/robots/fr3_duo/fr3_duo_cover/fr3_duo_cover.xacro" />
   <!--
     DEPRECATION NOTICE
@@ -53,7 +52,4 @@
       <origin xyz="0 0 0" rpy="0 0 0" />
   </xacro:mount>
-  <xacro:cover name="cover" parent="mount_link" inertials="${xacro.load_yaml('$(find franka_description)/robots/fr3_duo/fr3_duo_cover/inertials.yaml')}">
-      <origin xyz="0 0 0.068" rpy="0 0 0" />
-  </xacro:cover>
   <xacro:property name="number_of_robots" value = "2"/>
   <xacro:property name="arm_prefixes_list" value="${['left','right']}" />
@@ -83,5 +79,5 @@
                           joint_limits="${xacro.load_yaml('$(arg joint_limits_path)')}"
                           inertials="${xacro.load_yaml('$(arg inertials_path)')}"
-                          kinematics="${xacro.load_yaml('$(arg kinematics_path')}"
+                          kinematics="${xacro.load_yaml('$(arg kinematics_path)')}"
                           dynamics="${xacro.load_yaml('$(arg dynamics_path)')}"
                           accelerometer_config="${xacro.load_yaml('$(arg accelerometers_path)')}"

File: robots/fr3_duo/fr3_duo_fixed_structure.urdf.xacro (robot description, xacro)
@@ -3,5 +3,4 @@
   <xacro:include filename="$(find franka_description)/robots/common/franka_robot.xacro"/>
   <xacro:include filename="$(find franka_description)/robots/fr3_duo/fr3_duo_mount/fr3_duo_mount.xacro" />
-  <xacro:include filename="$(find franka_description)/robots/fr3_duo/fr3_duo_cover/fr3_duo_cover.xacro" />
   <link name="base">
   </link>
@@ -9,7 +8,3 @@
       <origin xyz="0 0 0" rpy="0 0 0" />
   </xacro:mount>
-  <xacro:arg name="cover_kinematics" default="$(find franka_description)/robots/fr3_duo/fr3_duo_cover/kinematics.yaml"/>
-  <xacro:cover name="cover" parent="mount_link" inertials="${xacro.load_yaml('$(find franka_description)/robots/fr3_duo/fr3_duo_cover/inertials.yaml')}">
-      <origin xyz="0 0 0.068" rpy="0 0 0" />
-  </xacro:cover>
 </robot>

File: robots/fr3_duo/fr3_duo_mount/fr3_duo_mount.xacro (robot description, xacro)
@@ -6,10 +6,22 @@
       <visual>
         <geometry>
-          <mesh filename="package://franka_description/meshes/robot_arms/fr3_duo/mount/visual/fr3_duo_mount.dae"/>
+          <mesh filename="package://franka_description/meshes/accessories/fr3_duo_mount/visual/fr3_duo_mount.dae"/>
+        </geometry>
+      </visual>
+      <visual>
+        <origin xyz="0 0 0.068" rpy="0 0 0" />
+        <geometry>
+          <mesh filename="package://franka_description/meshes/accessories/fr3_duo_mount/visual/fr3_duo_cover.dae"/>
         </geometry>
       </visual>
       <collision>
         <geometry>
-          <mesh filename="package://franka_description/meshes/robot_arms/fr3_duo/mount/collision/fr3_duo_mount.stl"/>
+          <mesh filename="package://franka_description/meshes/accessories/fr3_duo_mount/collision/fr3_duo_mount.stl"/>
+        </geometry>
+      </collision>
+      <collision>
+        <origin xyz="0 0 0.068" rpy="0 0 0" />
+        <geometry>
+          <mesh filename="package://franka_description/meshes/accessories/fr3_duo_mount/collision/fr3_duo_cover.stl"/>
         </geometry>
       </collision>
