Commit message: fr3

File: fr3_urdfs/fr3_cobot_pump.urdf (robot description, URDF)
Before this commit: robot fr3, 26 links, 25 joints
Links:
- removed link fr3_hand
- removed link fr3_hand_tcp
- removed link fr3_leftfinger
- removed link fr3_rightfinger
- added link fr3_cobot_pump, mass 1.01; collision mesh filename=./meshes/robot_ee/cobot_pump/collision/cobot_pump.stl; visual mesh filename=./meshes/robot_ee/cobot_pump/visual/cobot_pump.dae
- added link fr3_cobot_pump_tcp
Joints:
- removed joint fr3_finger_joint1
- removed joint fr3_finger_joint2
- removed joint fr3_hand_joint
- removed joint fr3_hand_tcp_joint
- added joint fr3_cobot_pump_joint: type fixed, parent fr3_link8, child fr3_cobot_pump, origin xyz=0 0 0 rpy=0 0 -0.7853981633974483
- added joint fr3_cobot_pump_tcp_joint: type fixed, parent fr3_cobot_pump, child fr3_cobot_pump_tcp, origin xyz=0 0 0.1034 rpy=0 0 0
