Commit message: fr3

File: fr3_urdfs/fr3_franka_hand.urdf (robot description, URDF)
Before this commit: robot fr3, 24 links, 23 joints
Links:
- removed link fr3_cobot_pump
- removed link fr3_cobot_pump_tcp
- added link fr3_hand, mass 0.6544; collision mesh filename=./meshes/robot_ee/franka_hand_white/collision/hand.stl; visual mesh filename=./meshes/robot_ee/franka_hand_white/visual/hand.dae
- added link fr3_hand_tcp
- added link fr3_leftfinger, mass 0.0291; collision box size=17.5e-3 15.2e-3 18.5e-3; collision box size=17.5e-3 7e-3 23.5e-3
- added link fr3_rightfinger, mass 0.0291; collision box size=17.5e-3 15.2e-3 18.5e-3; collision box size=17.5e-3 7e-3 23.5e-3
Joints:
- removed joint fr3_cobot_pump_joint
- removed joint fr3_cobot_pump_tcp_joint
- added joint fr3_finger_joint1: type prismatic, parent fr3_hand, child fr3_leftfinger, origin xyz=0 0 0.0584 rpy=0 0 0, axis 0 1 0, limit lower=0.0 upper=0.04 effort=100 velocity=0.2
- added joint fr3_finger_joint2: type prismatic, parent fr3_hand, child fr3_rightfinger, origin xyz=0 0 0.0584 rpy=0 0 3.141592653589793, axis 0 1 0, limit lower=0.0 upper=0.04 effort=100 velocity=0.2, mimic joint=fr3_finger_joint1
- added joint fr3_hand_joint: type fixed, parent fr3_link8, child fr3_hand, origin xyz=0 0 0 rpy=0 0 -0.7853981633974483
- added joint fr3_hand_tcp_joint: type fixed, parent fr3_hand, child fr3_hand_tcp, origin xyz=0 0 0.1034 rpy=0 0 0

Commit message: fr3

File: fr3_urdfs/fr3_franka_hand.urdf (robot description, URDF)
Before this commit: robot fr3, 26 links, 25 joints
Links:
- removed link fr3_hand
- removed link fr3_hand_tcp
- removed link fr3_leftfinger
- removed link fr3_rightfinger
- added link hand, mass 0.6544; collision mesh filename=./meshes/robot_ee/franka_hand_white/collision/hand.stl; visual mesh filename=./meshes/robot_ee/franka_hand_white/visual/hand.dae
- added link hand_tcp
- added link leftfinger, mass 0.0291; collision box size=17.5e-3 15.2e-3 18.5e-3; collision box size=17.5e-3 7e-3 23.5e-3
- added link rightfinger, mass 0.0291; collision box size=17.5e-3 15.2e-3 18.5e-3; collision box size=17.5e-3 7e-3 23.5e-3
Joints:
- removed joint fr3_finger_joint1
- removed joint fr3_finger_joint2
- removed joint fr3_hand_joint
- removed joint fr3_hand_tcp_joint
- added joint finger_joint1: type prismatic, parent hand, child leftfinger, origin xyz=0 0 0.0584 rpy=0 0 0, axis 0 1 0, limit lower=0.0 upper=0.04 effort=100 velocity=0.2
- added joint finger_joint2: type prismatic, parent hand, child rightfinger, origin xyz=0 0 0.0584 rpy=0 0 3.141592653589793, axis 0 1 0, limit lower=0.0 upper=0.04 effort=100 velocity=0.2, mimic joint=finger_joint1
- added joint hand_joint: type fixed, parent link8, child hand, origin xyz=0 0 0 rpy=0 0 -0.7853981633974483
- added joint hand_tcp_joint: type fixed, parent hand, child hand_tcp, origin xyz=0 0 0.1034 rpy=0 0 0

Commit message: urdf

File: fr3_urdfs/fr3_franka_hand.urdf (robot description, URDF)
Before this commit: robot fr3, 26 links, 25 joints
Links:
- link hand: geometry collision mesh filename=hand.stl; visual mesh filename=hand.dae
- link leftfinger: geometry collision box size=17.5e-3 15.2e-3 18.5e-3; collision box size=17.5e-3 7e-3 23.5e-3
- link link0: geometry collision mesh filename=link0.stl; visual mesh filename=link0.dae
- link link1: geometry collision mesh filename=link1.stl; visual mesh filename=link1.dae
- link link2: geometry collision mesh filename=link2.stl; visual mesh filename=link2.dae
- link link3: geometry collision mesh filename=link3.stl; visual mesh filename=link3.dae
- link link4: geometry collision mesh filename=link4.stl; visual mesh filename=link4.dae
- link link5: geometry collision mesh filename=link5.stl; visual mesh filename=link5.dae
- link link6: geometry collision mesh filename=link6.stl; visual mesh filename=link6.dae
- link link7: geometry collision mesh filename=link7.stl; visual mesh filename=link7.dae
- link rightfinger: geometry collision box size=17.5e-3 15.2e-3 18.5e-3; collision box size=17.5e-3 7e-3 23.5e-3
